File: Laser_Array_CPU.brd (EAGLE design)
At the start: 160 x 100 mm, 81 parts, among them IC1 PIC24FJ64GA004, J3 22-23-2021, M1 MOTOR, U2 MAX6817, U3 LP2985-28DBVTE4, X1 22-23-2031, X2 22-23-2041, X4 22-23-2041

Commit message: commit before push
Parts:
- added S16, S17, S18, S19: TC74, Mine:SOT23-5L
Changed lines of the file:
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@@
 <element name="S14" library="Mine" package="22-23-2021" value="TOGGLE_SPST" x="11.43" y="-1068.07"/>
 <element name="S15" library="Mine" package="22-23-2021" value="TOGGLE_SPST" x="11.43" y="-1088.39"/>
+<element name="S16" library="Mine" package="SOT23-5L" value="TC74" x="2.54" y="-1102.36"/>
+<element name="S17" library="Mine" package="SOT23-5L" value="TC74" x="2.54" y="-1109.98"/>
+<element name="S18" library="Mine" package="SOT23-5L" value="TC74" x="2.54" y="-1117.6"/>
+<element name="S19" library="Mine" package="SOT23-5L" value="TC74" x="2.54" y="-1125.22"/>
 </elements>
 <signals>
