File: Laser_Array_CPU.sch (EAGLE design)
At the start: 81 parts, among them IC1 PIC24FJ64GA004, J3 22-23-2021, M1 MOTOR, U2 MAX6817, U3 LP2985-28DBVTE4, X1 22-23-2031, X2 22-23-2041, X4 22-23-2041

Commit message: commit before push
Parts:
- added S16, S17, S18, S19: TC74, Mine:TC74
Changed lines of the file:
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@@
 <part name="SUPPLY28" library="supply2" deviceset="GND" device=""/>
 <part name="SUPPLY29" library="supply2" deviceset="GND" device=""/>
+<part name="S16" library="Mine" deviceset="TC74" device=""/>
+<part name="S17" library="Mine" deviceset="TC74" device=""/>
+<part name="S18" library="Mine" deviceset="TC74" device=""/>
+<part name="S19" library="Mine" deviceset="TC74" device=""/>
 </parts>
 <sheets>
@@
 <attribute name="VALUE" x="280.035" y="45.085" size="1.778" layer="96"/>
 </instance>
+<instance part="S16" gate="G$1" x="335.28" y="55.88"/>
+<instance part="S17" gate="G$1" x="358.14" y="38.1"/>
+<instance part="S18" gate="G$1" x="335.28" y="20.32"/>
+<instance part="S19" gate="G$1" x="358.14" y="2.54"/>
 </instances>
 <busses>
