File: Laser_Array.brd (EAGLE design)
At the start: 160 x 100 mm, 85 parts, among them IC1 PIC24FJ64GA004, J3 22-23-2021, M1 MOTOR, U2 MAX6817, U3 LP2985-28DBVTE4, X1 22-23-2031, X2 22-23-2041, X4 22-23-2041

Commit message: added temp sensors
Parts:
- added LED26: (no value), Mine:LED5MM
- added R10: 330, rcl:R0805
- added S20, S21, S22, S23, S24, S25, S26, S27: TC74, Mine:SOT23-5L
Connections:
- new net N$29: LED26.K, R10.2
- net GND: now also R10.1, S16.2, S17.2, S18.2, S19.2, S20.2, S21.2, S22.2, S23.2, S24.2, S25.2, S26.2, S27.2
- net LASOUT: now also LED26.A
- net SCLK1: now also S16.4, S17.4, S18.4, S19.4, S20.4, S21.4, S22.4, S23.4, S24.4, S25.4, S26.4, S27.4
- net SDA1: now also S16.5, S17.5, S18.5, S19.5, S20.5, S21.5, S22.5, S23.5, S24.5, S25.5, S26.5, S27.5
- net VDD: now also S16.3, S17.3, S18.3, S19.3, S20.3, S21.3, S22.3, S23.3, S24.3, S25.3, S26.3, S27.3
