File: Laser_Array.sch (EAGLE design)
At the start: 85 parts, among them IC1 PIC24FJ64GA004, J3 22-23-2021, M1 MOTOR, U2 MAX6817, U3 LP2985-28DBVTE4, X1 22-23-2031, X2 22-23-2041, X4 22-23-2041

Commit message: added temp sensors
Parts:
- added LED26: (no value), Mine:LEDA5MM
- added R10: 330, rcl:R-US_R0805
- added S20, S21, S22, S23, S24, S25, S26, S27: TC74, Mine:TC74
Connections:
- new net N$29: LED26.C, R10.2
- net GND: now also R10.1, S16.GND, S17.GND, S18.GND, S19.GND, S20.GND, S21.GND, S22.GND, S23.GND, S24.GND, S25.GND, S26.GND, S27.GND
- net LASOUT: now also LED26.A
- net SCLK1: now also S16.SCLK, S17.SCLK, S18.SCLK, S19.SCLK, S20.SCLK, S21.SCLK, S22.SCLK, S23.SCLK, S24.SCLK, S25.SCLK, S26.SCLK, S27.SCLK
- net SDA1: now also S16.SDA, S17.SDA, S18.SDA, S19.SDA, S20.SDA, S21.SDA, S22.SDA, S23.SDA, S24.SDA, S25.SDA, S26.SDA, S27.SDA
- net VDD: now also S16.VDD, S17.VDD, S18.VDD, S19.VDD, S20.VDD, S21.VDD, S22.VDD, S23.VDD, S24.VDD, S25.VDD, S26.VDD, S27.VDD
Other:
- note added: "Laser Array"
- note added: "TS1"
- note added: "TS10"
- note added: "TS11"
- note added: "TS12"
- note added: "TS2"
- note added: "TS3"
- note added: "TS4"
- note added: "TS5"
- note added: "TS6"
- note added: "TS7"
- note added: "TS8"
- note added: "TS9"
- note added: "Temperature Array"

Commit message: added temp sensors as breakout board
Parts:
- removed S20, S21, S22, S23, S24, S26, S27: TC74, Mine:TC74
- added C12: 10nF, rcl:C-USC0805
- added C13: 2.2uF, rcl:C-USC0805
- added C16: 1uF, rcl:C-USC0805
- added R11, R12, R13, R14, R15, R16, R17, R18, R19, R20, R21, R22, R23, R24, R25, R26, R27, R28, R29, R30, R31, R32, R33, R34, R35, R36, R37, R38: 4.7k, rcl:R-US_M0805
- added S28, S29, S30, S31, S32, S33, S34: TC74, Mine:TC74
- added U1, U4: TCA9548A, Mine:TCA9548A
- added U5: LP2985A-33DBVTE4, Texas Instruments_By_element14_Batch_1:LP2985A-33DBVTE4
- added X5: 22-23-2041, Mine:22-23-2041
- added X6: 22-23-2031, Mine:22-23-2031
Connections:
- new net !RESET: IC1.TDO, R25.2, R30.2, U1.!RESET, U4.!RESET, X2-4.S, X5-4.S
- new net A0: IC1.RB4, U1.A0, U4.A0, X2-3.S, X5-3.S
- new net N$30: IC1.RA4
- new net N$35: C12.1, U5.BYPASS
- new net SC0: R12.2, S25.SCLK, U4.SC0
- new net SC1: R16.2, S28.SCLK, U4.SC1
- new net SC10: R36.2, S18.SCLK, U1.SC2
- new net SC11: R38.2, S19.SCLK, U1.SC3
- new net SC2: R18.2, S29.SCLK, U4.SC2
- new net SC3: R20.2, S30.SCLK, U4.SC3
- new net SC4: R22.2, S31.SCLK, U4.SC4
- new net SC5: R24.2, S32.SCLK, U4.SC5
- new net SC6: R27.2, S33.SCLK, U4.SC6
- new net SC7: R29.2, S34.SCLK, U4.SC7
- new net SC8: R32.2, S16.SCLK, U1.SC0
- new net SC9: R34.2, S17.SCLK, U1.SC1
- new net SCK1: X2-1.S, X5-1.S
- new net SD0: R11.2, S25.SDA, U4.SD0
- new net SD1: R15.2, S28.SDA, U4.SD1
- new net SD10: R35.2, S18.SDA, U1.SD2
- new net SD11: R37.2, S19.SDA, U1.SD3
- new net SD2: R17.2, S29.SDA, U4.SD2
- new net SD3: R19.2, S30.SDA, U4.SD3
- new net SD4: R21.2, S31.SDA, U4.SD4
- new net SD5: R23.2, S32.SDA, U4.SD5
- new net SD6: R26.2, S33.SDA, U4.SD6
- new net SD7: R28.2, S34.SDA, U4.SD7
- new net SD8: R31.2, S16.SDA, U1.SD0
- new net SD9: R33.2, S17.SDA, U1.SD1
- new net VTS: C13.1, S16.GND, S17.GND, S18.GND, S19.GND, S25.GND, S28.GND, S29.GND, S30.GND, S31.GND, S32.GND, S33.GND, S34.GND, U5.VOUT
- net +12V: now also C16.1, U5.ON/OFF, U5.VIN, X6-2.S
- net GND: now also C12.2, C13.2, C16.2, S16.VDD, S17.VDD, S18.VDD, S19.VDD, S25.VDD, S28.VDD, S29.VDD, S30.VDD, S31.VDD, S32.VDD, S33.VDD, S34.VDD, U1.A1, U1.A2, U1.GND, U4.A1, U4.A2, U4.GND, U5.GND, X6-1.S; no longer S16.GND, S17.GND, S18.GND, S19.GND, S20.GND, S21.GND, S22.GND, S23.GND, S24.GND, S25.GND, S26.GND, S27.GND, X2-2.S
- net SCLK1: now also R14.1, U1.SCL, U4.SCL; no longer S16.SCLK, S17.SCLK, S18.SCLK, S19.SCLK, S20.SCLK, S21.SCLK, S22.SCLK, S23.SCLK, S24.SCLK, S25.SCLK, S26.SCLK, S27.SCLK, X2-3.S
- net SDA1: now also R13.1, U1.SDA, U4.SDA, X2-2.S, X5-2.S; no longer S16.SDA, S17.SDA, S18.SDA, S19.SDA, S20.SDA, S21.SDA, S22.SDA, S23.SDA, S24.SDA, S25.SDA, S26.SDA, S27.SDA, X2-4.S
- net VDD: now also R11.1, R12.1, R13.2, R14.2, R15.1, R16.1, R17.1, R18.1, R19.1, R20.1, R21.1, R22.1, R23.1, R24.1, R25.1, R26.1, R27.1, R28.1, R29.1, R30.1, R31.1, R32.1, R33.1, R34.1, R35.1, R36.1, R37.1, R38.1, U1.VDD, U4.VDD, X6-3.S; no longer S16.VDD, S17.VDD, S18.VDD, S19.VDD, S20.VDD, S21.VDD, S22.VDD, S23.VDD, S24.VDD, S25.VDD, S26.VDD, S27.VDD, X2-1.S
Other:
- note added: "!RST"
- note added: "+12V"
- note added: "3.3V"
- note added: "A0"
- note added: "SCLK1"
- note added: "Signal Header"
- note added: "TS0"
- note added: "Temp Sensor Breakout Board Header"
- note added: "To Temp Sensor Breakout Board"
- note removed: "SLKL1"
- note removed: "TS12"
- moved on the sheet: C10, C11, R6, R7, X2-1, X2-2, X2-3, X2-4, X4-1, X4-2, X4-3, X4-4

Commit message: commit on surface 2
Other:
- note added: "Altered on Surface"
Changed lines of the file:
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@@
 <?xml version="1.0" encoding="utf-8"?>
 <!DOCTYPE eagle SYSTEM "eagle.dtd">
-<eagle version="7.7.0">
+<eagle version="7.6.0">
 <drawing>
 <settings>
@@
 <setting verticaltext="up"/>
 </settings>
-<grid distance="0.1" unitdist="inch" unit="inch" style="lines" multiple="1" display="yes" altdistance="0.01" altunitdist="inch" altunit="inch"/>
+<grid distance="0.1" unitdist="inch" unit="inch" style="lines" multiple="1" display="no" altdistance="0.01" altunitdist="inch" altunit="inch"/>
 <layers>
 <layer number="1" name="Top" color="4" fill="1" visible="no" active="no"/>
@@
 <text x="322.58" y="-109.22" size="1.778" layer="91">TS10</text>
 <text x="393.7" y="-109.22" size="1.778" layer="91">TS11</text>
+<text x="-76.2" y="101.6" size="1.778" layer="91">Altered on Surface</text>
 </plain>
 <instances>

Commit message: altered for surface
Other:
- note added: "Altered again on laptob."
Changed lines of the file:
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@@
 <?xml version="1.0" encoding="utf-8"?>
 <!DOCTYPE eagle SYSTEM "eagle.dtd">
-<eagle version="7.6.0">
+<eagle version="7.7.0">
 <drawing>
 <settings>
@@
 <text x="393.7" y="-109.22" size="1.778" layer="91">TS11</text>
 <text x="-76.2" y="101.6" size="1.778" layer="91">Altered on Surface</text>
+<text x="-78.74" y="96.52" size="1.778" layer="91">Altered again on laptob.</text>
 </plain>
 <instances>

Commit message: added MCU decoupling capacitor C17
Parts:
- added C17: 0.1uF, rcl:C-USC0805
Connections:
- net GND: now also C17.2
- net VDD: now also C17.1
Changed lines of the file:
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@@
 <part name="R37" library="rcl" deviceset="R-US_" device="M0805" value="4.7k"/>
 <part name="R38" library="rcl" deviceset="R-US_" device="M0805" value="4.7k"/>
+<part name="C17" library="rcl" deviceset="C-US" device="C0805" value="0.1uF"/>
 </parts>
 <sheets>
@@
 <attribute name="VALUE" x="369.57" y="-127.762" size="1.778" layer="96"/>
 </instance>
+<instance part="C17" gate="G$1" x="-12.7" y="-50.8" smashed="yes" rot="R90">
+<attribute name="NAME" x="-12.192" y="-45.847" size="1.778" layer="95" rot="R180"/>
+<attribute name="VALUE" x="-9.398" y="-54.483" size="1.778" layer="96" rot="R180"/>
+</instance>
 </instances>
 <busses>
@@
 <segment>
 <pinref part="IC1" gate="G$1" pin="AVDD"/>
-<wire x1="0" y1="-35.56" x2="0" y2="-53.34" width="0.1524" layer="91"/>
+<wire x1="0" y1="-35.56" x2="0" y2="-43.18" width="0.1524" layer="91"/>
+<wire x1="0" y1="-43.18" x2="0" y2="-53.34" width="0.1524" layer="91"/>
 <wire x1="0" y1="-53.34" x2="0" y2="-73.66" width="0.1524" layer="91"/>
 <wire x1="0" y1="-73.66" x2="-12.7" y2="-73.66" width="0.1524" layer="91"/>
@@
 <wire x1="25.4" y1="-53.34" x2="0" y2="-53.34" width="0.1524" layer="91"/>
 <junction x="0" y="-53.34"/>
+<pinref part="C17" gate="G$1" pin="1"/>
+<wire x1="-15.24" y1="-50.8" x2="-17.78" y2="-50.8" width="0.1524" layer="91"/>
+<wire x1="-17.78" y1="-50.8" x2="-17.78" y2="-43.18" width="0.1524" layer="91"/>
+<wire x1="-17.78" y1="-43.18" x2="0" y2="-43.18" width="0.1524" layer="91"/>
+<junction x="0" y="-43.18"/>
 </segment>
 <segment>
@@
 <wire x1="-50.8" y1="-63.5" x2="-2.54" y2="-63.5" width="0.1524" layer="91"/>
 <junction x="-2.54" y="-63.5"/>
-</segment>
-<segment>
+<pinref part="C17" gate="G$1" pin="2"/>
+<wire x1="-7.62" y1="-50.8" x2="-2.54" y2="-50.8" width="0.1524" layer="91"/>
+</segment>
+<segment>

Commit message: added CS and DC to schematic
Connections:
- net N$8 renamed DC
Changed lines of the file:
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@@
 </segment>
 </net>
-<net name="N$8" class="0">
+<net name="DC" class="0">
 <segment>
 <pinref part="J2" gate="-3" pin="S"/>
@@
 <pinref part="IC1" gate="G$1" pin="RB12"/>
 <wire x1="-38.1" y1="-10.16" x2="-35.56" y2="-10.16" width="0.1524" layer="91"/>
+<wire x1="-38.1" y1="-20.32" x2="-38.1" y2="-22.86" width="0.1524" layer="91"/>
+<junction x="-38.1" y="-20.32"/>
+<label x="-38.1" y="-22.86" size="1.778" layer="95" rot="R180" xref="yes"/>
 </segment>
 </net>
@@
 <segment>
 <pinref part="J2" gate="-6" pin="S"/>
-<wire x1="-88.9" y1="-27.94" x2="-38.1" y2="-27.94" width="0.1524" layer="91"/>
+<wire x1="-88.9" y1="-27.94" x2="-83.82" y2="-27.94" width="0.1524" layer="91"/>
 <pinref part="IC1" gate="G$1" pin="TMS"/>
+<wire x1="-83.82" y1="-27.94" x2="-38.1" y2="-27.94" width="0.1524" layer="91"/>
 <wire x1="-12.7" y1="-35.56" x2="-12.7" y2="-38.1" width="0.1524" layer="91"/>
 <wire x1="-12.7" y1="-38.1" x2="-38.1" y2="-38.1" width="0.1524" layer="91"/>
 <wire x1="-38.1" y1="-38.1" x2="-38.1" y2="-27.94" width="0.1524" layer="91"/>
+<wire x1="-83.82" y1="-27.94" x2="-83.82" y2="-30.48" width="0.1524" layer="91"/>
+<junction x="-83.82" y="-27.94"/>
+<label x="-83.82" y="-30.48" size="1.778" layer="95" rot="R270" xref="yes"/>
 </segment>
 </net>

Commit message: Started CPU Board
Parts:
- removed J2: (no value), Mine:22-23-2061
- added C19, C20: 10nF, rcl:C-USC0805
- added SV1: (no value), con-lstb:MA12-2
- added SV2: (no value), con-lstb:MA17-2W
Connections:
- removed net N$30: IC1.RA4
- removed net SCK1: X2-1.S, X5-1.S
- removed net SCLK1: IC1.RB8, R14.1, S3.SCLK, U1.SCL, U4.SCL
- new net SCL1: IC1.RB8, R14.1, S3.SCLK
- new net SCL2: IC1.RB3, U1.SCL, U4.SCL, X2-1.S, X5-1.S
- new net SDA2: IC1.RB2, U1.SDA, U4.SDA, X2-2.S, X5-2.S
- net A0: no longer IC1.RB4, U1.A0, U4.A0
- net CS: now also SV1.9; no longer J2-6.S
- net DC: now also SV1.11; no longer J2-3.S
- net ENCDR_A: now also IC1.RC3; no longer IC1.RB3
- net ENCDR_B: now also IC1.RC4; no longer IC1.RB2
- net GND: now also C19.2, C20.2, SV2.25, U4.A0; no longer J2-2.S
- net MOSI: now also SV2.9; no longer J2-5.S
- net SCLK: now also SV2.11; no longer J2-4.S
- net SDA1: no longer U1.SDA, U4.SDA, X2-2.S, X5-2.S
- net VDD: now also C19.1, C20.1, SV2.29, U1.A0; no longer J2-1.S
Other:
- moved on the sheet: C1, R13, R14, R25

Commit message: temperture sensor board & CPU board complete
Parts:
- removed S28, S29, S30, S31, S32, S33, S34: TC74, Mine:TC74
- removed X4: 22-23-2041, Mine:22-23-2041
- removed X6: 22-23-2031, Mine:22-23-2031
- added C21: 10nF, rcl:C-USC0805
- added C22: 2.2uF, rcl:C-USC0805
- added C23: 470uF, rcl:CPOL-USF
- added D3, D4, D6: 641-1014-6-ND, adafruit:DIODESOD-123
- added D5: S10M-TPMSCT_ND, Mine:S10M-TPMSCT_ND
- added D7, D8: LL4148FSCT-ND, semicon-smd-ipc:D-SOD-80
- added J2, J4, J5, J7, J8, J9: 22-23-2021, Mine:22-23-2021
- added J6: (no value), Mine:RJ_25
- added R39: 4.7k, rcl:R-US_M0805
- added S20, S21, S22, S23, S24, S26, S27: TOGGLE_SPST, Mine:TOGGLE_SPST
- added X3, X7, X8, X9: 22-23-2041, Mine:22-23-2041
- C1, C2: value 0.1uF -> 10F; device rcl:C-USC0805 -> rcl:CPOL-USE5-10.5
- C10: value 10nF -> 10uF; device rcl:C-USC0805 -> Mine:CAP3X3
- C11: value 10nF -> 18pF
- C12, C9: value 10nF -> 0.1uF
- C13: value 2.2uF -> 18pF
- C16: value 1uF -> 10nF
- C17: value 0.1uF -> 2.2uF
- C18: value 2.2uF -> 1uF
- C3: value 10uF -> 0.1uF
- C4: value 18pF -> 0.1uF
- C5: value 18pF -> 10uF
- C6: value 0.1uF -> 10nF
- C7: value 10uF -> 10nF; device Mine:CAP3X3 -> rcl:C-USC0805
- D1: value LL4148FSCT-ND -> S10M-TPMSCT_ND; device semicon-smd-ipc:D-SOD-80 -> Mine:S10M-TPMSCT_ND
- D2: value LL4148FSCT-ND -> 641-1014-6-ND; device semicon-smd-ipc:D-SOD-80 -> adafruit:DIODESOD-123
- J1: value (none) -> 22-23-2021; device Mine:RJ_25 -> Mine:22-23-2021
- LED2: value LED3MM -> (none); device Mine:LED3MM -> Mine:LEDA5MM
- LED26: value (none) -> LED3MM; device Mine:LEDA5MM -> Mine:LED3MM
- Q1: device adafruit:CRYSTALSM49 -> Mine:QS5U34CT-ND_MOSFET_N_CHANNEL
- Q4: device Mine:QS5U34CT-ND_MOSFET_N_CHANNEL -> adafruit:CRYSTALSM49
- R1: value 10k -> 10R, 5W; device rcl:R-US_R0805 -> Mine:RESISTOR5W
- R10: value 330 -> 4.7k; device rcl:R-US_R0805 -> rcl:R-US_M0805
- R11: value 4.7k -> 330; device rcl:R-US_M0805 -> rcl:R-US_R0805
- R12: value 4.7k -> 220k
- R13: value 4.7k -> 200k; device rcl:R-US_M0805 -> rcl:R-TRIMM3224X
- R2: value 100k -> 10k
- R4: value 220k -> 100k; device rcl:R-US_M0805 -> rcl:R-US_R0805
- R5: value 200k -> 10k; device rcl:R-TRIMM3224X -> rcl:R-US_M0805
- R7: device rcl:R-US_M0805 -> rcl:R-US_R0805
- R8: value 10k -> 4.7k; device rcl:R-US_R0805 -> rcl:R-US_M0805
- S1: value TACT_PB -> (none); device Mine:TACT_PB -> Mine:DPDT_TOGGLE
- S10, S11, S12, S13, S14, S15, S4, S5, S6, S7, S8, S9: value TOGGLE_SPST -> TC74; device Mine:TOGGLE_SPST -> Mine:TC74
- S16, S17, S18, S19, S25: value TC74 -> TOGGLE_SPST; device Mine:TC74 -> Mine:TOGGLE_SPST
- S2: value (none) -> TACT_PB; device Mine:DPDT_TOGGLE -> Mine:TACT_PB
- SV1: device con-lstb:MA12-2 -> con-lstb:MA17-2W
- SV2: device con-lstb:MA17-2W -> con-lstb:MA12-2
- U1: value TCA9548A -> MAX6817; device Mine:TCA9548A -> Mine:MAX6817
- U2: value MAX6817 -> LP2985-28DBVTE4; device Mine:MAX6817 -> Texas Instruments_By_element14_Batch_1:LP2985-28DBVTE4
- U3: value LP2985-28DBVTE4 -> TCA9548A; device Texas Instruments_By_element14_Batch_1:LP2985-28DBVTE4 -> Mine:TCA9548A
- X1: value 22-23-2031 -> 22-23-2041; device Mine:22-23-2031 -> Mine:22-23-2041
Connections:
- removed net A0: X2-3.S, X5-3.S
- removed net ENSW: U2.IN1, X4-4.S
- removed net N$14: U2.OUT1
- new net CHGOUTA: IC1.RC6, J9-1.S
- new net CHGOUTB: IC1.RC7, J9-2.S
- new net ENSW_I: U1.IN1, X3-4.S
- new net ENSW_O: IC1.RB15, U1.OUT1
- new net N$30: J1-1.S, LED1.A
- new net N$31: C19.1, U5.BYPASS
- new net N$32: J2-2.S, Q1.D
- new net N$33: D3.C, D4.A, R1.2
- new net N$34: J7-1.S, Q3.D
- new net N$36: C1.-, C2.+
- new net N$37: C1.+, D5.A, R1.1
- new net N$8: D1.A, D2.C
- new net VLASER: D1.C, RLY12.P, X1-4.S, X2-4.S, X8-4.S, X9-4.S
- net !RESET: now also R14.2, R15.2, U3.!RESET, X8-3.S, X9-3.S; no longer R25.2, R30.2, U1.!RESET, X2-4.S, X5-4.S
- net +12V: now also C18.1, J2-1.S, R12.2, U2.ON/OFF, U2.VIN, X2-2.S, X5-3.S, X7-3.S; no longer C16.1, LED1.A, R4.2, U3.ON/OFF, U3.VIN, X1-2.S, X6-2.S
- net +12V_TB: now also D6.C, RLY2.+12V, X1-2.S
- net CHGA: now also J8-1.S; no longer J3-1.S
- net CHGB: now also J8-2.S; no longer J3-2.S
- net CS: now also SV2.9; no longer SV1.9
- net DC: now also SV2.11; no longer SV1.11
- net ENCDR_A: now also C7.1, R5.1, X3-3.S; no longer C11.1, R7.1, X4-3.S
- net ENCDR_B: now also C6.1, X3-2.S; no longer C10.1, X4-2.S
- net EXFAN: now also Q2.G, R4.1; no longer Q3.G, R3.1
- net GND: now also C10.-, C2.-, C21.2, C22.2, C23.-, C7.2, C9.1, D8.A, J3-2.S, J4-2.S, J5-2.S, J6.4, J7-2.S, LED26.C, LED8.C, Q1.S, R11.1, R13.A, R4.2, RLY2.GND, S1.P, S10.GND, S11.GND, S12.GND, S13.GND, S14.GND, S15.GND, S2.1, S4.GND, S5.GND, S6.GND, S7.GND, S8.GND, S9.GND, SV1.25, U3.A0, U3.A1, U3.A2, X1-3.S, X2-3.S, X3-1.S, X5-4.S, X7-4.S; no longer C1.1, C10.2, C2.2, C7.-, C9.2, D2.A, J1.4, LED14.C, LED2.C, Q4.S, R10.1, R2.2, R5.A, S1.1, S16.VDD, S17.VDD, S18.VDD, S19.VDD, S2.P, S25.VDD, S28.VDD, S29.VDD, S30.VDD, S31.VDD, S32.VDD, S33.VDD, S34.VDD, SV2.25, U1.A1, U1.A2, U4.A0, X1-1.S, X4-1.S, X6-1.S
- net LASOUT: now also LED2.A, RLY2.NC1; no longer LED26.A, RLY2.COM1
- net LASRLY: now also Q3.G; no longer Q4.G
- net MOSI: now also SV1.9; no longer SV2.9
- net N$1: now also C10.+, J6.6, R7.2, S2.2; no longer C7.+, J1.6, R1.2, S1.2
- net N$10: now also U1.OUT2; no longer U2.OUT2
- net N$11: now also J1-2.S; no longer Q2.D
- net N$12: now also J3-1.S, Q2.D; no longer M1.+, Q3.D
- net N$13: now also R13.E; no longer R5.E
- net N$15: now also D6.A, J5-1.S; no longer Q4.D
- net N$16: now also LED17.A, S18.O; no longer LED18.A, S6.O
- net N$17: now also RLY2.COM1, S16.I, S17.I, S18.I, S19.I, S20.I, S21.I, S22.I, S23.I, S24.I, S25.I, S26.I, S27.I; no longer RLY2.NC1, S10.I, S11.I, S12.I, S13.I, S14.I, S15.I, S4.I, S5.I, S6.I, S7.I, S8.I, S9.I
- net N$18: now also LED15.A, LED3.A, S16.O; no longer LED16.A, LED2.A, S4.O
- net N$19: now also LED16.A, LED9.A, S17.O; no longer LED15.A, LED3.A, S5.O
- net N$2: now also C5.1; no longer C3.1
- net N$20: now also LED10.A, LED18.A, S19.O; no longer LED21.A, LED5.A, S7.O
- net N$21: now also LED19.A, LED5.A, S20.O; no longer LED17.A, LED6.A, S9.O
- net N$22: now also LED11.A, LED20.A, S21.O; no longer LED25.A, LED7.A, S10.O
- net N$23: now also LED21.A, LED6.A, S22.O; no longer LED13.A, LED23.A, S11.O
- net N$24: now also LED22.A, S23.O; no longer LED19.A, S12.O
- net N$25: now also LED23.A, LED7.A, S24.O; no longer LED11.A, LED14.A, S14.O
- net N$26: now also LED13.A, LED24.A, S25.O; no longer LED10.A, LED20.A, S15.O
- net N$27: now also LED25.A, LED8.A, S26.O; no longer LED22.A, LED9.A, S8.O
- net N$28: now also LED14.A, LED26.A, S27.O; no longer LED24.A, LED8.A, S13.O
- net N$29: now also LED2.C, R11.2; no longer LED26.C, R10.2
- net N$3: now also J6.1; no longer J1.1
- net N$35: now also J4-1.S, M1.+; no longer C12.1, U5.BYPASS
- net N$4: now also J6.2; no longer J1.2
- net N$5: now also J6.3; no longer J1.3
- net N$55: now also U2.BYPASS; no longer U3.BYPASS
- net N$6: now also C11.1, Q4.1; no longer C5.1, Q1.1
- net N$7: now also C13.1, Q4.2; no longer C4.1, Q1.2
- net N$9: now also R2.1, S1.S, U1.IN2; no longer R8.1, S2.S, U2.IN2
- net ONLED: now also Q1.G, R3.1; no longer Q2.G, R2.1
- net SC0: now also R22.2, S4.SCLK, U3.SC0; no longer R12.2, S25.SCLK, U4.SC0
- net SC1: now also R34.2, S10.SCLK, U3.SC1; no longer R16.2, S28.SCLK, U4.SC1
- net SC10: now also R27.2, S9.SCLK, U4.SC2; no longer R36.2, S18.SCLK, U1.SC2
- net SC11: now also R39.2, S15.SCLK, U4.SC3; no longer R38.2, S19.SCLK, U1.SC3
- net SC2: now also R23.2, S5.SCLK, U3.SC2; no longer R18.2, S29.SCLK, U4.SC2
- net SC3: now also R35.2, S11.SCLK, U3.SC3; no longer R20.2, S30.SCLK, U4.SC3
- net SC4: now also R24.2, S6.SCLK, U3.SC4; no longer R22.2, S31.SCLK, U4.SC4
- net SC5: now also R36.2, S12.SCLK, U3.SC5; no longer R24.2, S32.SCLK, U4.SC5
- net SC6: now also R25.2, S7.SCLK, U3.SC6; no longer R27.2, S33.SCLK, U4.SC6
- net SC7: now also R37.2, S13.SCLK, U3.SC7; no longer R29.2, S34.SCLK, U4.SC7
- net SC8: now also R26.2, S8.SCLK, U4.SC0; no longer R32.2, S16.SCLK, U1.SC0
- net SC9: now also R38.2, S14.SCLK, U4.SC1; no longer R34.2, S17.SCLK, U1.SC1
- net SCL1: now also R10.1; no longer R14.1
- net SCL2: now also U3.SCL, X8-1.S, X9-1.S; no longer U1.SCL, X2-1.S, X5-1.S
- net SCLK: now also SV1.11; no longer SV2.11
- net SD0: now also R16.2, S4.SDA, U3.SD0; no longer R11.2, S25.SDA, U4.SD0
- net SD1: now also R28.2, S10.SDA, U3.SD1; no longer R15.2, S28.SDA, U4.SD1
- net SD10: now also R21.2, S9.SDA, U4.SD2; no longer R35.2, S18.SDA, U1.SD2
- net SD11: now also R33.2, S15.SDA, U4.SD3; no longer R37.2, S19.SDA, U1.SD3
- net SD2: now also S5.SDA, U3.SD2; no longer S29.SDA, U4.SD2
- net SD3: now also R29.2, S11.SDA, U3.SD3; no longer R19.2, S30.SDA, U4.SD3
- net SD4: now also R18.2, S6.SDA, U3.SD4; no longer R21.2, S31.SDA, U4.SD4
- net SD5: now also R30.2, S12.SDA, U3.SD5; no longer R23.2, S32.SDA, U4.SD5
- net SD6: now also R19.2, S7.SDA, U3.SD6; no longer R26.2, S33.SDA, U4.SD6
- net SD7: now also R31.2, S13.SDA, U3.SD7; no longer R28.2, S34.SDA, U4.SD7
- net SD8: now also R20.2, S8.SDA, U4.SD0; no longer R31.2, S16.SDA, U1.SD0
- net SD9: now also R32.2, S14.SDA, U4.SD1; no longer R33.2, S17.SDA, U1.SD1
- net SDA1: now also R8.1; no longer R13.1
- net SDA2: now also U3.SDA, X8-2.S, X9-2.S; no longer U1.SDA, X2-2.S, X5-2.S
- net VDD: now also C12.1, C21.1, C3.1, C4.1, C9.2, D4.C, D5.C, J6.5, R10.2, R14.1, R2.2, R39.1, R5.2, R7.1, SV1.29, U3.VDD, U4.A0, X5-1.S, X7-1.S; no longer C1.2, C17.1, C19.1, C2.1, C6.1, J1.5, R1.1, R11.1, R12.1, R13.2, R14.2, R7.2, S3.VDD, SV2.29, U1.A0, U2.VDD, X1-3.S, X6-3.S
- net VDD_TB: now also D2.A, D3.A, X1-1.S, X2-1.S; no longer RLY12.P
- net VIN1: now also C16.1, D7.A, D8.C, R12.1, R13.S; no longer C9.1, D1.A, D2.C, R4.1, R5.S
- net VRR: now also C17.1, D7.C, U2.VOUT; no longer C18.1, D1.C, U3.VOUT
- net VTS: now also C22.1, C23.+, S10.VDD, S11.VDD, S12.VDD, S13.VDD, S14.VDD, S15.VDD, S3.VDD, S4.VDD, S5.VDD, S6.VDD, S7.VDD, S8.VDD, S9.VDD, X5-2.S, X7-2.S; no longer C13.1, S16.GND, S17.GND, S18.GND, S19.GND, S25.GND, S28.GND, S29.GND, S30.GND, S31.GND, S32.GND, S33.GND, S34.GND
Other:
- note added: "(on PCU Brd)"
- note added: "(on TEMP SENSOR Brd)"
- note added: "***"
- note added: "*** Across contact screws."
- note added: "+12V_TB"
- note added: "3.1V"
- note added: "4.4V"
- note added: "CHGOUTLEDA"
- note added: "CHGOUTLEDB"
- note added: "Ext Fan Header"
- note added: "LASER ON LED"
- note added: "Laser Relay Header"
- note added: "Note: 3V illumination voltage"
- note added: "ON LED Header"
- note added: "VDD_TB"
- note added: "VLASER"
- note added: "VTS"
- note removed: "A0"
- note removed: "Signal Header"
- moved on the sheet: C11, C12, C13, C16, C17, C18, C19, C20, C3, C4, C5, C6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
