File: Laser_Charger.brd (EAGLE design)
At the start: 160 x 100 mm, 22 parts, among them P1 12V/3V_DC/DC_CONVERTER, X1 6ESRM-P

Commit message: temperture sensor board & CPU board complete
Parts:
- CHG1, CHG2: device Mine:SLA_CHARGER -> Mine:22-23-2101
- moved CHG2 356.4 mm to (19.0, -284.0)
- moved CHG1 320.0 mm to (19.0, -268.0)
- moved RLY1 249.2 mm to (16.0, -224.0)
- moved RLY2 148.0 mm to (16.0, -246.0)
Connections:
- net +12V: now also RLY2.9; no longer RLY2.2
- net +BAT: now also RLY1.3; no longer RLY1.7
- net -BAT: now also RLY1.2, RLY2.3; no longer RLY1.10, RLY2.7
- net GND: now also RLY2.12, RLY2.7; no longer RLY2.8, RLY2.9
- net N$1: now also RLY2.4; no longer RLY2.10
- net N$10: now also RLY2.8; no longer RLY2.12
- net N$11: now also CHG1.10, RLY1.5; no longer CHG1.1, RLY1.3
- net N$12: now also CHG1.7; no longer CHG1.8
- net N$13: now also CHG2.3; no longer CHG2.4
- net N$14: now also CHG2.7; no longer CHG2.8
- net N$15: now also CHG2.8, CHG2.9, RLY1.8; no longer CHG2.2, CHG2.3, RLY1.12
- net N$17: now also CHG2.10, RLY1.7; no longer CHG2.1, RLY1.9
- net N$3: now also RLY1.9; no longer RLY1.2
- net N$4: now also RLY1.10; no longer RLY1.5
- net N$5: now also RLY1.11; no longer RLY1.8
- net N$6: now also CHG1.8, CHG1.9; no longer CHG1.2, CHG1.3
- net N$7: now also CHG1.3; no longer CHG1.4
- net N$8: now also RLY1.12; no longer RLY1.11
- net N$9: now also RLY2.2; no longer RLY2.4
- net STAT1: now also CHG1.4; no longer CHG1.7
- net STAT2: now also CHG2.4; no longer CHG2.7
- net VCC: now also CHG1.1, CHG1.2, CHG2.1, CHG2.2, RLY2.5; no longer CHG1.10, CHG1.9, CHG2.10, CHG2.9, RLY2.3
- net VDD: now also RLY2.10; no longer RLY2.5
