File: Laser_Charger.sch (EAGLE design)
At the start: 22 parts, among them P1 12V/3V_DC/DC_CONVERTER, X1 6ESRM-P

Commit message: temperture sensor board & CPU board complete
Other:
- note added: "CHARGE Relay"
- note added: "POWER Relay"
