File: Laser_Array_CPU_V1.1.brd (EAGLE design)
At the start: 102.3 x 109.6 mm, 68 parts, among them IC1 PIC24FJ64GA004, J1 MA16-2, J3 22-23-2021, J4 22-23-2021, J8 22-23-2021, J9 22-23-2021, U1 MAX6817, U2 LP2985-28DBVTE4, U3 LP2985A-33DBVTE4, X1 22-23-2031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

Commit message: Finished Laser_Array_V1.2
Parts:
- removed U3: LP2985A-33DBVTE4, Texas Instruments_By_element14_Batch_1:SOT95P280X145-5N
- removed X4: 87758-0616, Mine:87758-0616
- added D10, D6, D9: (no value), Mine:DO214AC
- added J2: (no value), Mine:RJ11-NO_SHIELD
- added RLY1: RELAY_SPST_1A, Mine:RELAY_SPST_1A
- added U4: LP2985-50DBVR, Texas Instruments_By_element14_Batch_1:SOT95P280X145-5N
- D2, D3: value 641-1014-6-ND -> S10M-TPMSCT_ND; device adafruit:SOD-123 -> Mine:S10M-TPMSCT-ND
- D4: value 641-1014-6-ND -> (none); device adafruit:SOD-123 -> Mine:DO214AC
- D5: value S10M-TPMSCT_ND -> (none); device Mine:S10M-TPMSCT-ND -> Mine:DO214AC
- moved D5 91.0 mm to (-28.2, 14.5), turned to 0 degrees
- moved D4 81.4 mm to (-28.2, 18.5), turned to 0 degrees
- moved D3 75.5 mm to (-29.5, 30.2), turned to 0 degrees
- moved D2 62.5 mm to (-20.1, 30.2), turned to 0 degrees
- moved C10 2.05 mm to (44.8, 87.2)
- moved C7 1.11 mm to (47.5, 87.2), turned to 90 degrees
- moved C4 1.02 mm to (30.3, 84.1)
- moved R16 0.51 mm to (30.7, 81.3)
Connections:
- removed net N$34: J8.1, Q3.5
- removed net N$35: C15.1, U3.4
- removed net N$5: IC1.21, X4.3
- new net N$12: D6.A, J4.2, Q2.5
- new net N$13: D9.A, J8.2, Q3.5
- new net N$14: C1.1, J1.29, RLY1.1
- new net N$15: C15.1, U4.4
- net +12V: now also D6.C, D9.C, J8.1, U4.1, U4.3; no longer U3.1, U3.3
- net GND: now also C1.2, J1.25, J2.4, U4.2; no longer J4.2, J8.2, U3.2, X4.4
- net N$1: now also J2.6; no longer X4.6
- net N$16: now also IC1.21, J2.3; no longer J4.1, Q2.5
- net N$4: now also J2.2; no longer X4.2
- net N$8: now also D10.A, RLY1.3; no longer C1.2, J1.25
- net VDD: now also D10.C, J2.5, RLY1.2, RLY1.4; no longer C1.1, J1.29, X4.5
- net VIN1: now also IC1.41; no longer IC1.19
- net VTS: now also U4.5; no longer U3.5
Routing:
- net N$34: track 128.3 -> 0.00 mm, vias 2 -> 0
- net N$16: track 68.7 -> 27.1 mm
- net N$5: track 30.4 -> 0.00 mm, vias 2 -> 0
- net N$1: track 99.3 -> 71.7 mm
- net N$4: track 56.2 -> 42.9 mm, vias 4 -> 2
- net N$8: track 11.6 -> 0.00 mm
- net VDD: track 259.5 -> 250.2 mm
- net N$3: track 7.60 -> 0.00 mm
- net N$33: track 15.5 -> 9.65 mm
- net GND: track 20.7 -> 25.4 mm, vias 12 -> 10
- net N$35: track 4.15 -> 0.00 mm
- net VDD_TB: track 11.0 -> 6.90 mm
- net VIN1: track 70.5 -> 67.0 mm
- net VTS: track 42.5 -> 39.7 mm
- net VLASER: track 67.8 -> 65.6 mm
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