File: Laser_Array_CPU_V1.2.brd (EAGLE design)
At the start: 102.3 x 109.6 mm, 72 parts, among them IC1 PIC24FJ64GA004, J1 MA16-2, J3 22-23-2021, J4 22-23-2021, J8 22-23-2021, J9 22-23-2021, U1 MAX6817, U2 LP2985-28DBVTE4, U4 LP2985-50DBVR, X1 22-23-2031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

Commit message: Finished Laser_Array_V1.2
Parts:
- moved D10 156.1 mm to (68.1, 109.5), turned to 180 degrees
- moved RLY1 135.5 mm to (68.1, 98.3), turned to 90 degrees
- moved D9 106.3 mm to (56.6, 70.4), turned to 180 degrees
- moved D6 97.8 mm to (49.0, 70.4), turned to 180 degrees
- moved D5 90.7 mm to (46.5, 66.0)
- moved J8 86.3 mm to (94.5, 80.9), turned to 90 degrees
- moved D4 85.9 mm to (46.5, 61.0)
- moved D3 76.0 mm to (45.5, 43.2), turned to 180 degrees
- moved D2 69.3 mm to (45.2, 53.6), turned to 270 degrees
- moved U4 37.6 mm to (19.8, 67.3)
- moved S1 16.5 mm to (94.6, 64.4)
- moved C10 8.64 mm to (41.2, 79.3)
- moved C7 6.23 mm to (42.0, 84.3), turned to 270 degrees
- moved J4 5.85 mm to (94.3, 88.4)
- moved C14 4.41 mm to (27.5, 61.0), turned to 90 degrees
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Connections:
- net +12V: now also J4.1
- net N$14: no longer C1.1
- net VDD: now also C1.1
Routing:
- net VIN1: track 67.0 -> 245.3 mm, vias 0 -> 6
- net +12V: track 298.2 -> 445.0 mm
- net N$12: track 0.00 -> 95.0 mm, vias 0 -> 2
- net N$13: track 0.00 -> 86.2 mm, vias 0 -> 2
- net N$4: track 0.00 -> 42.9 mm, vias 0 -> 2
- net N$14: track 0.00 -> 36.6 mm
- net N$8: track 0.00 -> 36.3 mm
- net VDD: track 244.7 -> 278.7 mm
- net N$1: track 65.5 -> 93.6 mm
- net N$9: track 82.8 -> 105.6 mm
- net N$33: track 9.65 -> 26.6 mm
- net VDD_TB: track 6.90 -> 19.8 mm
- net N$3: track 0.00 -> 6.14 mm
- net GND: track 25.4 -> 20.7 mm
- net N$15: track 0.00 -> 4.53 mm
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Other:
- board size 102.3 x 109.6 mm -> 104.1 x 109.6 mm
- board text added: "September 28, 1018 Terawatt Productions Inc."
- board text removed: "September 18, 1018 Terawatt Productions Inc."
