File: Laser_Array_CPU_V1.2.sch (EAGLE design)
At the start: 72 parts, among them IC1 PIC24FJ64GA004, J1 MA16-2, J3 22-23-2021, J4 22-23-2021, J8 22-23-2021, J9 22-23-2021, U1 MAX6817, U2 LP2985-28DBVTE4, U4 LP2985-50DBVR, X1 22-23-2031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

Commit message: Finished Laser_Array_V1.2
Connections:
- net +12V: now also J4-1.S
- net N$14: no longer C1.1
- net VDD: now also C1.1
Other:
- moved on the sheet: C1, D9, J2
Changed lines of the file:
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@@
 <attribute name="VALUE" x="-65.024" y="138.049" size="1.778" layer="96"/>
 </instance>
-<instance part="C1" gate="G$1" x="-134.62" y="40.64" smashed="yes">
-<attribute name="NAME" x="-133.604" y="41.275" size="1.778" layer="95"/>
-<attribute name="VALUE" x="-133.604" y="36.449" size="1.778" layer="96"/>
+<instance part="C1" gate="G$1" x="-139.7" y="40.64" smashed="yes">
+<attribute name="NAME" x="-136.144" y="41.275" size="1.778" layer="95"/>
+<attribute name="VALUE" x="-136.144" y="36.449" size="1.778" layer="96"/>
 </instance>
 <instance part="S1" gate="S" x="-101.6" y="111.76" smashed="yes" rot="R270">
@@
 <instance part="D5" gate="G$1" x="-83.82" y="-68.58" rot="R90"/>
 <instance part="D6" gate="G$1" x="-5.08" y="-33.02" rot="R90"/>
-<instance part="D9" gate="G$1" x="-5.08" y="-66.04" rot="R90"/>
+<instance part="D9" gate="G$1" x="-5.08" y="-68.58" rot="R90"/>
 <instance part="RLY1" gate="G$1" x="-127" y="71.12" smashed="yes" rot="MR180">
 <attribute name="PART" x="-125.73" y="76.2" size="1.778" layer="95" rot="MR180"/>
@@
 <instance part="D10" gate="G$1" x="-116.84" y="71.12" rot="MR90"/>
 <instance part="U4" gate="A" x="195.58" y="147.32"/>
-<instance part="J2" gate="G$1" x="60.96" y="5.08"/>
+<instance part="J2" gate="G$1" x="63.5" y="5.08"/>
 </instances>
 <busses>
@@
 <pinref part="J2" gate="G$1" pin="5"/>
 <wire x1="35.56" y1="2.54" x2="15.24" y2="2.54" width="0.1524" layer="91"/>
-<wire x1="55.88" y1="0" x2="35.56" y2="0" width="0.1524" layer="91"/>
+<wire x1="58.42" y1="0" x2="35.56" y2="0" width="0.1524" layer="91"/>
 <wire x1="35.56" y1="0" x2="35.56" y2="2.54" width="0.1524" layer="91"/>
 </segment>
@@
 <wire x1="-116.84" y1="78.74" x2="-127" y2="78.74" width="0.1524" layer="91"/>
 <junction x="-127" y="78.74"/>
+<pinref part="C1" gate="G$1" pin="1"/>
+<wire x1="-139.7" y1="43.18" x2="-139.7" y2="78.74" width="0.1524" layer="91"/>
+<wire x1="-139.7" y1="78.74" x2="-134.62" y2="78.74" width="0.1524" layer="91"/>
 </segment>
 </net>
@@
 </segment>
 <segment>
-<wire x1="7.62" y1="-35.56" x2="0" y2="-35.56" width="0.1524" layer="91"/>
+<wire x1="5.08" y1="-35.56" x2="0" y2="-35.56" width="0.1524" layer="91"/>
 <wire x1="0" y1="-35.56" x2="0" y2="-27.94" width="0.1524" layer="91"/>
 <wire x1="0" y1="-27.94" x2="-5.08" y2="-27.94" width="0.1524" layer="91"/>
@@
 <wire x1="-5.08" y1="-30.48" x2="-5.08" y2="-27.94" width="0.1524" layer="91"/>
 <junction x="-5.08" y="-27.94"/>
+<pinref part="J4" gate="-1" pin="S"/>
 </segment>
 <segment>
@@
 <pinref part="D9" gate="G$1" pin="C"/>
 <wire x1="-5.08" y1="-60.96" x2="-10.16" y2="-60.96" width="0.1524" layer="91"/>
-<wire x1="-5.08" y1="-63.5" x2="-5.08" y2="-60.96" width="0.1524" layer="91"/>
+<wire x1="-5.08" y1="-66.04" x2="-5.08" y2="-60.96" width="0.1524" layer="91"/>
 <junction x="-5.08" y="-60.96"/>
 </segment>
@@
 <wire x1="7.62" y1="5.08" x2="12.7" y2="5.08" width="0.1524" layer="91"/>
 <pinref part="J2" gate="G$1" pin="4"/>
-<wire x1="55.88" y1="2.54" x2="40.64" y2="2.54" width="0.1524" layer="91"/>
+<wire x1="58.42" y1="2.54" x2="40.64" y2="2.54" width="0.1524" layer="91"/>
 <wire x1="40.64" y1="2.54" x2="40.64" y2="5.08" width="0.1524" layer="91"/>
 <wire x1="40.64" y1="5.08" x2="12.7" y2="5.08" width="0.1524" layer="91"/>
@@
 <segment>
 <pinref part="C1" gate="G$1" pin="2"/>
-<wire x1="-134.62" y1="35.56" x2="-134.62" y2="33.02" width="0.1524" layer="91"/>
-<wire x1="-134.62" y1="33.02" x2="-121.92" y2="33.02" width="0.1524" layer="91"/>
+<wire x1="-139.7" y1="35.56" x2="-139.7" y2="33.02" width="0.1524" layer="91"/>
+<wire x1="-139.7" y1="33.02" x2="-121.92" y2="33.02" width="0.1524" layer="91"/>
 <pinref part="J1" gate="G$1" pin="25"/>
 <pinref part="R14" gate="G$1" pin="2"/>
@@
 <junction x="35.56" y="-12.7"/>
 <pinref part="J2" gate="G$1" pin="6"/>
-<wire x1="55.88" y1="-2.54" x2="35.56" y2="-2.54" width="0.1524" layer="91"/>
+<wire x1="58.42" y1="-2.54" x2="35.56" y2="-2.54" width="0.1524" layer="91"/>
 <junction x="35.56" y="-2.54"/>
 </segment>
@@
 <wire x1="27.94" y1="20.32" x2="27.94" y2="17.78" width="0.1524" layer="91"/>
 <pinref part="J2" gate="G$1" pin="2"/>
-<wire x1="55.88" y1="7.62" x2="45.72" y2="7.62" width="0.1524" layer="91"/>
+<wire x1="58.42" y1="7.62" x2="45.72" y2="7.62" width="0.1524" layer="91"/>
 <wire x1="45.72" y1="7.62" x2="45.72" y2="17.78" width="0.1524" layer="91"/>
 <wire x1="45.72" y1="17.78" x2="27.94" y2="17.78" width="0.1524" layer="91"/>
@@
 <pinref part="D9" gate="G$1" pin="A"/>
 <wire x1="-5.08" y1="-73.66" x2="10.16" y2="-73.66" width="0.1524" layer="91"/>
-<wire x1="-5.08" y1="-68.58" x2="-5.08" y2="-73.66" width="0.1524" layer="91"/>
+<wire x1="-5.08" y1="-71.12" x2="-5.08" y2="-73.66" width="0.1524" layer="91"/>
 <junction x="-5.08" y="-73.66"/>
 </segment>
@@
 <wire x1="-134.62" y1="50.8" x2="-134.62" y2="66.04" width="0.1524" layer="91"/>
 <pinref part="RLY1" gate="G$2" pin="S"/>
-<pinref part="C1" gate="G$1" pin="1"/>
-<wire x1="-134.62" y1="43.18" x2="-134.62" y2="50.8" width="0.1524" layer="91"/>
-<junction x="-134.62" y="50.8"/>
-</segment>
-</net>
-<net name="N$19" class="0">
-<segment>
-<wire x1="256.54" y1="109.22" x2="256.54" y2="111.76" width="0.1524" layer="91"/>
 </segment>
 </net>
@@
 <wire x1="25.4" y1="20.32" x2="25.4" y2="15.24" width="0.1524" layer="91"/>
 <pinref part="J2" gate="G$1" pin="3"/>
-<wire x1="55.88" y1="5.08" x2="43.18" y2="5.08" width="0.1524" layer="91"/>
+<wire x1="58.42" y1="5.08" x2="43.18" y2="5.08" width="0.1524" layer="91"/>
 <wire x1="43.18" y1="5.08" x2="43.18" y2="15.24" width="0.1524" layer="91"/>
 <wire x1="43.18" y1="15.24" x2="25.4" y2="15.24" width="0.1524" layer="91"/>
