File: Laser_Array_CPU_V1.5.brd (EAGLE design)
At the start: 104.1 x 109.6 mm, 72 parts, among them IC1 PIC24FJ64GA004, J1 MA16-2, J3 22-23-2021, J4 22-23-2021, J8 22-23-2021, U1 MAX6817, U2 LP2985-28DBVTE4, U4 LP2985-50DBVR, X1 22-23-2031, X2 22-23-2041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

Commit message: Finished Laser_Array CPU Board V 1.5
Parts:
- removed C2, C3: 10F, rcl:E5-10,5
- removed D3: S10M-TPMSCT_ND, Mine:S10M-TPMSCT-ND
- removed U3: (no value), Mine:SOT223
- removed X1: 22-23-2031, Mine:22-23-2031
- added D1, D2: (no value), Mine:DO214AC
- added J5, J6: 22-23-2021, Mine:22-23-2021
- added Q6, Q7: (no value), Mine:SOT23-5L
- added R17: 100k, rcl:R0805
- added U5: VOLTAGE_REG_APD1154ADL, Mine:SOIC8
- C23: value 4.7uF -> 1uF
- R15, R9: value 4.7k -> 2.2k
- R3: value 2R2, 5W -> 100k; device Mine:RESISTOR5W -> rcl:R0805
- moved S3 42.5 mm to (71.5, 50.2)
- moved R7 42.3 mm to (76.8, 48.2)
- moved R6 41.0 mm to (76.8, 51.9), turned to 0 degrees
- moved R3 26.2 mm to (71.1, 81.8), turned to 90 degrees
- moved C23 11.6 mm to (30.7, 55.4), turned to 270 degrees
- moved D6 6.49 mm to (54.6, 67.1)
- moved C17 5.59 mm to (33.1, 68.2)
- moved C22 5.47 mm to (43.7, 55.4), turned to 270 degrees
- moved D9 5.08 mm to (61.7, 70.4)
Connections:
- removed net CHGOUTA: IC1.2, X1.1
- removed net CHGOUTB: IC1.3, X1.2
- removed net N$36: C2.-, C3.+
- removed net N$37: C2.+, R3.1
- removed net VDD_TB: C23.1, D3.C, R3.2, U3.1
- new net HEAT_RLY: IC1.2, Q6.1, R3.1
- new net N$17: D2.A, J6.2, Q7.5
- new net N$3: C23.1, U5.6, U5.7, X2.1
- new net N$5: D1.A, J5.2, Q6.5
- new net SPARE: IC1.3, Q7.1, R17.1
- net +12V: now also D1.C, D2.C, J5.1, J6.1
- net GND: now also Q6.2, Q7.2, R17.2, R3.2, U5.1, U5.3, U5.4, U5.5, U5.8; no longer C3.-, U3.2, U3.4, X1.3
- net VDD: now also U5.2; no longer U3.3
- net VLASER: no longer D3.A, X2.1
Routing:
- net CHGOUTA: track 106.9 -> 0.00 mm
- net CHGOUTB: track 104.9 -> 0.00 mm
- net +12V: track 445.0 -> 527.4 mm, vias 0 -> 2
- net N$5: track 0.00 -> 54.2 mm
- net HEAT_RLY: track 0.00 -> 51.3 mm
- net SPARE: track 0.00 -> 50.8 mm
- net N$17: track 0.00 -> 50.7 mm
- net VTS: track 41.5 -> 87.4 mm
- net SCL1: track 47.1 -> 91.2 mm
- net SDA1: track 43.1 -> 75.3 mm
- net VDD_TB: track 30.3 -> 0.00 mm
- net VDD: track 288.8 -> 318.4 mm, vias 10 -> 8
- net VLASER: track 82.1 -> 57.7 mm
- net N$3: track 0.00 -> 14.7 mm
- net N$37: track 9.07 -> 0.00 mm
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Other:
- board text added: "Heat"
- board text added: "March 4, 1019 Terawatt Productions Inc."
- board text added: "Spare"
- board text removed: "CHGOUT"
- board text removed: "November 19, 1018 Terawatt Productions Inc."
