File: Laser_Array_CPU_V1.5.sch (EAGLE design)
At the start: 71 parts, among them IC1 PIC24FJ64GA004, J1 MA16-2, J3 22-23-2021, J4 22-23-2021, J8 22-23-2021, U1 MAX6817, U2 LP2985-28DBVTE4, U4 LP2985-50DBVR, X1 22-23-2031, X2 22-23-2041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

Commit message: Finished Laser_Array CPU Board V 1.5
Parts:
- removed C2, C3: 10F, rcl:CPOL-USE5-10.5
- removed D3: S10M-TPMSCT_ND, Mine:S10M-TPMSCT_ND
- removed U3: (no value), Mine:V_REG_3.0V_1.0A
- removed X1: 22-23-2031, Mine:22-23-2031
- added D1, D2: (no value), Mine:DIODE_GENPURP_1A_100V
- added J5, J6: 22-23-2021, Mine:22-23-2021
- added Q6, Q7: (no value), Mine:QS5U34CT-ND_MOSFET_N_CHANNEL
- added R17: 100k, rcl:R-US_R0805
- added SJ1: (no value), jumper:SJ
- added U5: VOLTAGE_REG_APD1154ADL, Mine:VOLTAGE_REG_APD1154ADL
- C23: value 4.7uF -> 1uF
- R15, R9: value 4.7k -> 2.2k
- R3: value 2R2, 5W -> 100k; device Mine:RESISTOR5W -> rcl:R-US_R0805
Connections:
- removed net CHGOUTA: IC1.RC6, X1-1.S
- removed net CHGOUTB: IC1.RC7, X1-2.S
- removed net N$36: C2.-, C3.+
- removed net N$37: C2.+, R3.1
- removed net VDD_TB: C23.1, D3.C, R3.2, U3.P$1
- new net HEAT_RLY: IC1.RC6, Q6.G, R3.1
- new net N$17: D2.A, J6-2.S, Q7.D
- new net N$3: C23.1, U5.VCONT, U5.VIN, X2-1.S
- new net N$5: D1.A, J5-2.S, Q6.D
- new net SPARE: IC1.RC7, Q7.G, R17.1
- net +12V: now also D1.C, D2.C, J5-1.S, J6-1.S
- net GND: now also Q6.S, Q7.S, R17.2, R3.2, U5.GND, U5.NC, U5.NC1, U5.NC2, U5.PLC; no longer C3.-, U3.P$2, U3.P$4, X1-3.S
- net VDD: now also U5.VOUT; no longer U3.P$3
- net VIN1: now also SJ1.1, SJ1.2
- net VLASER: no longer D3.A, X2-1.S
Other:
- note added: "3.3V Reg"
- note added: "5.0 V"
- note added: "Heater Relay Coil"
- note added: "Spare"
- note removed: "4.5V"
- note removed: "CHGOUTLEDA"
- note removed: "CHGOUTLEDB"
- moved on the sheet: C21, C22, C23, D7, D8, R10, R11, R3, X4-1, X4-2, X4-3
